File: project/Basic_STM32_Bluepill.kicad_pcb (KiCad board)
At the start: 2 copper layers, 43 x 34 mm, 33 parts, among them J1 Conn_01x04_Pin, J2 Conn_01x04_Pin, J3 USB_B_Micro, J4 Conn_01x04_Pin, SW1 SW_SPDT, U1 AMS1117-3.3, U2 STM32F103C8T6, Y1 16 MHz

Commit message: First draft of changes
Added the RPi style connector and an extra for remaining pins.
Parts:
- removed G***: LOGO, LOGO
- removed the J3 at (171.9, 91.7)
- added C6: 100n, Capacitor_SMD:C_0402_1005Metric, F.Cu at (188.2, 95.3)
- added J4: USB_C_Receptacle_USB2.0, Connector_USB:USB_C_Receptacle_GCT_USB4105-xx-A_16P_TopMnt_Horizontal, F.Cu at (192.7, 89.7)
- added R10: 5K1, Resistor_SMD:R_0402_1005Metric, F.Cu at (188.3, 81.4)
- added R11: 5K1, Resistor_SMD:R_0402_1005Metric, F.Cu at (188.3, 83.4)
- added R2: 1k5, Resistor_SMD:R_0402_1005Metric, F.Cu at (188.3, 73.4)
- added R3: 1k5, Resistor_SMD:R_0402_1005Metric, F.Cu at (188.3, 75.4)
- added R8: 10K, Resistor_SMD:R_0402_1005Metric, F.Cu at (188.3, 79.4)
- added R9: 10K, Resistor_SMD:R_0402_1005Metric, F.Cu at (188.3, 77.4)
- J1: value Conn_01x04_Pin -> THD-20-R; footprint Connector_PinHeader_2.54mm:PinHeader_1x04_P2.54mm_Vertical -> Connector_PinHeader_2.54mm:PinHeader_2x20_P2.54mm_Vertical
- J2: value Conn_01x04_Pin -> THD-10-R; footprint Connector_PinHeader_2.54mm:PinHeader_1x04_P2.54mm_Vertical -> Connector_PinHeader_2.54mm:PinHeader_2x10_P2.54mm_Vertical
- U2: value STM32F103C8T6 -> STM32L475RGT7; footprint Package_QFP:LQFP-48_7x7mm_P0.5mm -> Package_QFP:LQFP-64_10x10mm_P0.5mm
- moved J2 62.6 mm to (217.0, 80.2), turned to 0 degrees
- moved J1 46.5 mm to (182.0, 74.7), turned to 0 degrees
- renumbered C9 to C10, C10 to C11, C11 to C12, C12 to C13, C13 to C14, C5 to C3, C3 to C4, C4 to C5, C6 to C7, C7 to C8, C8 to C9, J4 to J3, R2 to R4, R3 to R5, R4 to R6, R5 to R7
Connections:
- J1 pad 2: /I2C2_SCL -> VBUS
- J1 pad 4: GND -> VBUS
- J2 pad 2: /USART1_TX -> +3.3V
- J2 pad 3: /USART1_RX -> /PC15
- J2 pad 4: GND -> /PB3
- R4 pad 1: /I2C2_SCL -> /I2C1_SCL
- R5 pad 1: /I2C2_SDA -> /I2C1_SDA
- U2 pad 10: unconnected-(U2-PA0-Pad10) -> /SPI2_MISO
- U2 pad 11: unconnected-(U2-PA1-Pad11) -> /SPI2_MOSI
- U2 pad 12: unconnected-(U2-PA2-Pad12) -> GND
- U2 pad 13: unconnected-(U2-PA3-Pad13) -> +3.3V
- U2 pad 14: unconnected-(U2-PA4-Pad14) -> /PA0
- U2 pad 15: unconnected-(U2-PA5-Pad15) -> /GPIO18
- U2 pad 16: unconnected-(U2-PA6-Pad16) -> /USART2_TX
- U2 pad 17: unconnected-(U2-PA7-Pad17) -> /USART2_RX
- U2 pad 18: unconnected-(U2-PB0-Pad18) -> GND
- U2 pad 19: unconnected-(U2-PB1-Pad19) -> +3.3V
- U2 pad 2: unconnected-(U2-PC13-Pad2) -> /GPIO24
- U2 pad 20: unconnected-(U2-PB2-Pad20) -> /PA4
- U2 pad 21: /I2C2_SCL -> /SPI1_SCK
- U2 pad 22: /I2C2_SDA -> /SPI1_MISO
- U2 pad 23: GND -> /SPI1_MOSI
- U2 pad 24: +3.3V -> GND
- U2 pad 25: unconnected-(U2-PB12-Pad25) -> GND
- U2 pad 26: unconnected-(U2-PB13-Pad26) -> /PB0
- U2 pad 27: unconnected-(U2-PB14-Pad27) -> /PB1
- U2 pad 28: unconnected-(U2-PB15-Pad28) -> /PB2
- U2 pad 29: unconnected-(U2-PA8-Pad29) -> /SPI2_SCK
- U2 pad 3: unconnected-(U2-PC14-Pad3) -> /GPIO23
- U2 pad 30: unconnected-(U2-PA9-Pad30) -> /I2C2_SDA
- U2 pad 31: unconnected-(U2-PA10-Pad31) -> GND
- U2 pad 32: /USB_D- -> +3.3V
- U2 pad 33: /USB_D+ -> /PB12
- U2 pad 34: /SWDIO -> /I2C2_SCL
- U2 pad 35: GND -> /PB14
- U2 pad 36: +3.3V -> /PB15
- U2 pad 37: /SWCLK -> GND
- U2 pad 38: unconnected-(U2-PA15-Pad38) -> /GPIO26
- U2 pad 39: unconnected-(U2-PB3-Pad39) -> /GPIO16
- U2 pad 4: unconnected-(U2-PC15-Pad4) -> /PC15
- U2 pad 40: unconnected-(U2-PB4-Pad40) -> /GPIO12
- U2 pad 41: unconnected-(U2-PB5-Pad41) -> /PA8
- U2 pad 44: /BOOT0 -> /USB_D-
- U2 pad 45: unconnected-(U2-PB8-Pad45) -> /USB_D+
- U2 pad 46: unconnected-(U2-PB9-Pad46) -> /SWDIO
- U2 pad 48: +3.3V -> +3.3VA
- U2 pad 9: +3.3VA -> GND
Routing:
- net /USB_D-: track 12.7 -> 0.00 mm
- net /USART1_TX: track 9.26 -> 22.0 mm
- net /I2C2_SDA: track 10.3 -> 0.00 mm
- net /I2C1_SDA: track 0.00 -> 10.3 mm
